File: 8Bit-audio-v2/8Bit-audio-7524-axelb-v2.brd (EAGLE design)
At the start: 77.4 x 38.1 mm, 21 parts, among them IC1 LM358 or MCP6022, IC4 AD7524LN, X1 AUX 3,5mm

Commit message: New footprints
Parts:
- C1, C2, C6: device rcl:E5-5 -> myLbr:E2,5-7
- moved C6 6.35 mm to (52.1, 26.7)
- moved C2 2.54 mm to (40.6, 14.0)
- moved C1 1.36 mm to (32.2, 22.9)
Connections:
- net AUX: now also C6.-1
- net GND: now also C1.-1
- net N$3: now also C2.-1
Routing:
- net AUX: track 18.9 -> 26.5 mm
- net OUTB: track 34.9 -> 28.2 mm
- net N$5: track 31.5 -> 30.3 mm
Changed lines of the file:
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@@
 </autorouter>
 <elements>
-<element name="C1" library="rcl" library_urn="urn:adsk.eagle:library:334" package="E5-5" package3d_urn="urn:adsk.eagle:package:23367/2" value="100µ" x="31.75" y="21.59" smashed="yes" rot="R270">
-<attribute name="NAME" x="33.02" y="19.05" size="1.27" layer="25" ratio="10" rot="R270"/>
-<attribute name="POPULARITY" value="6" x="-10.16" y="-10.16" size="1.778" layer="27" rot="R270" display="off"/>
-<attribute name="SPICEPREFIX" value="C" x="-10.16" y="-10.16" size="1.778" layer="27" rot="R270" display="off"/>
-<attribute name="VALUE" x="29.21" y="19.05" size="1.27" layer="21" ratio="10" rot="R270"/>
+<element name="C1" library="myLbr" package="E2,5-7" value="100µ" x="32.22625" y="22.86" smashed="yes" rot="R270">
+<attribute name="NAME" x="33.49625" y="20.32" size="1.27" layer="25" ratio="10" rot="R270"/>
+<attribute name="POPULARITY" value="0" x="-9.68375" y="-8.89" size="1.778" layer="27" rot="R270" display="off"/>
+<attribute name="SPICEPREFIX" value="C" x="-9.68375" y="-8.89" size="1.778" layer="27" rot="R270" display="off"/>
+<attribute name="VALUE" x="29.68625" y="20.32" size="1.27" layer="21" ratio="10" rot="R270"/>
 </element>
 <element name="IC1" library="linear" library_urn="urn:adsk.eagle:library:262" package="DIL08" package3d_urn="urn:adsk.eagle:package:16409/2" value="LM358 or MCP6022" x="40.64" y="22.86" smashed="yes" rot="R270">
@@
 <attribute name="VALUE" x="32.385" y="10.5156" size="1.27" layer="21" ratio="10" rot="R270"/>
 </element>
-<element name="C2" library="rcl" library_urn="urn:adsk.eagle:library:334" package="E5-5" package3d_urn="urn:adsk.eagle:package:23367/2" value="1µ" x="38.1" y="13.97" smashed="yes" rot="R180">
-<attribute name="NAME" x="37.465" y="10.795" size="1.27" layer="21" ratio="10" rot="R180"/>
-<attribute name="POPULARITY" value="6" x="38.1" y="13.97" size="1.778" layer="27" rot="R180" display="off"/>
-<attribute name="SPICEPREFIX" value="C" x="38.1" y="13.97" size="1.778" layer="27" rot="R180" display="off"/>
-<attribute name="VALUE" x="40.005" y="10.795" size="1.27" layer="21" ratio="10" rot="R180"/>
+<element name="C2" library="myLbr" package="E2,5-7" value="1µ" x="40.64" y="13.97" smashed="yes" rot="R180">
+<attribute name="NAME" x="40.005" y="10.795" size="1.27" layer="21" ratio="10" rot="R180"/>
+<attribute name="POPULARITY" value="0" x="40.64" y="13.97" size="1.778" layer="27" rot="R180" display="off"/>
+<attribute name="SPICEPREFIX" value="C" x="40.64" y="13.97" size="1.778" layer="27" rot="R180" display="off"/>
+<attribute name="VALUE" x="42.545" y="10.795" size="1.27" layer="21" ratio="10" rot="R180"/>
 </element>
 <element name="R3" library="rcl" library_urn="urn:adsk.eagle:library:334" package="0207/10" package3d_urn="urn:adsk.eagle:package:23491/2" value="10k" x="53.34" y="7.62" smashed="yes">
@@
 <attribute name="VALUE" x="41.56075" y="10.06475" size="1.27" layer="21" ratio="10" rot="R270"/>
 </element>
-<element name="C6" library="rcl" library_urn="urn:adsk.eagle:library:334" package="E5-5" package3d_urn="urn:adsk.eagle:package:23367/2" value="100µ" x="58.42" y="26.67" smashed="yes">
-<attribute name="NAME" x="55.245" y="29.845" size="1.27" layer="21" ratio="10"/>
-<attribute name="POPULARITY" value="6" x="58.42" y="26.67" size="1.778" layer="27" display="off"/>
-<attribute name="SPICEPREFIX" value="C" x="58.42" y="26.67" size="1.778" layer="27" display="off"/>
-<attribute name="VALUE" x="57.785" y="29.845" size="1.27" layer="21" ratio="10"/>
+<element name="C6" library="myLbr" package="E2,5-7" value="100µ" x="52.07" y="26.67" smashed="yes">
+<attribute name="NAME" x="48.895" y="29.845" size="1.27" layer="21" ratio="10"/>
+<attribute name="POPULARITY" value="0" x="52.07" y="26.67" size="1.778" layer="27" display="off"/>
+<attribute name="SPICEPREFIX" value="C" x="52.07" y="26.67" size="1.778" layer="27" display="off"/>
+<attribute name="VALUE" x="51.435" y="29.845" size="1.27" layer="21" ratio="10"/>
 </element>
 <element name="R6" library="myLbr" package="POT_3RP/1610N" value="10k" x="71.12" y="11.43" smashed="yes" rot="R90">
@@
 <vertex x="77.47" y="0"/>
 </polygon>
+<contactref element="C1" pad="-1"/>
 </signal>
 <signal name="AUX">
@@
 <wire x1="64.69" y1="22.94" x2="63.5" y2="24.13" width="0.254" layer="16"/>
 <wire x1="63.5" y1="24.13" x2="63.5" y2="26.67" width="0.254" layer="16"/>
+<contactref element="C6" pad="-1"/>
 <wire x1="63.5" y1="26.67" x2="63.5" y2="31.75" width="0.254" layer="16"/>
-<wire x1="60.96" y1="26.67" x2="63.5" y2="26.67" width="0.254" layer="16"/>
+<wire x1="53.34" y1="26.67" x2="55.88" y2="26.67" width="0.254" layer="16"/>
+<wire x1="55.88" y1="26.67" x2="63.5" y2="26.67" width="0.254" layer="16"/>
 </signal>
 <signal name="D7">
@@
 <wire x1="48.26" y1="25.4" x2="48.26" y2="22.86" width="0.254" layer="1"/>
 <wire x1="48.26" y1="22.86" x2="45.72" y2="20.32" width="0.254" layer="1"/>
-<wire x1="35.56" y1="13.97" x2="33.02" y2="13.97" width="0.254" layer="1"/>
 <wire x1="45.72" y1="20.32" x2="40.64" y2="20.32" width="0.254" layer="1"/>
 <wire x1="40.64" y1="20.32" x2="39.37" y2="19.05" width="0.254" layer="1"/>
-<wire x1="39.37" y1="19.05" x2="39.37" y2="17.78" width="0.254" layer="1"/>
-<wire x1="39.37" y1="17.78" x2="35.56" y2="13.97" width="0.254" layer="1"/>
-<wire x1="48.26" y1="7.62" x2="39.37" y2="7.62" width="0.254" layer="1"/>
-<wire x1="39.37" y1="7.62" x2="35.56" y2="11.43" width="0.254" layer="1"/>
-<wire x1="35.56" y1="11.43" x2="35.56" y2="13.97" width="0.254" layer="1"/>
+<wire x1="39.37" y1="19.05" x2="39.37" y2="13.97" width="0.254" layer="1"/>
+<wire x1="48.26" y1="7.62" x2="40.64" y2="7.62" width="0.254" layer="1"/>
+<wire x1="40.64" y1="7.62" x2="39.37" y2="8.89" width="0.254" layer="1"/>
+<wire x1="39.37" y1="8.89" x2="39.37" y2="13.97" width="0.254" layer="1"/>
+<contactref element="C2" pad="-1"/>
+<wire x1="39.37" y1="13.97" x2="36.83" y2="13.97" width="0.254" layer="1"/>
+<wire x1="36.83" y1="13.97" x2="33.02" y2="13.97" width="0.254" layer="1"/>
 </signal>
 <signal name="N$6">
@@
 <contactref element="C6" pad="+"/>
 <wire x1="44.45" y1="24.13" x2="49.53" y2="24.13" width="0.254" layer="16"/>
-<wire x1="49.53" y1="24.13" x2="52.07" y2="26.67" width="0.254" layer="16"/>
+<wire x1="49.53" y1="24.13" x2="50.8" y2="25.4" width="0.254" layer="16"/>
 <wire x1="44.45" y1="21.59" x2="44.45" y2="24.13" width="0.254" layer="1"/>
-<wire x1="52.07" y1="26.67" x2="55.88" y2="26.67" width="0.254" layer="16"/>
+<wire x1="50.8" y1="25.4" x2="50.8" y2="26.67" width="0.254" layer="16"/>
 <contactref element="JP5" pad="1"/>
-<wire x1="55.88" y1="30.1625" x2="53.0225" y2="33.02" width="0.3048" layer="16"/>
-<wire x1="53.0225" y1="33.02" x2="50.8" y2="33.02" width="0.3048" layer="16"/>
-<wire x1="55.88" y1="26.67" x2="55.88" y2="30.1625" width="0.3048" layer="16"/>
+<wire x1="50.8" y1="33.02" x2="50.8" y2="26.67" width="0.3048" layer="16"/>
 <contactref element="C4" pad="2"/>
 <contactref element="C4" pad="3"/>
-<wire x1="55.88" y1="26.67" x2="55.88" y2="19.05" width="0.254" layer="1"/>
 <wire x1="55.88" y1="19.05" x2="53.34" y2="19.05" width="0.254" layer="1"/>
+<wire x1="50.8" y1="26.67" x2="50.8" y2="25.4" width="0.254" layer="1"/>
+<wire x1="50.8" y1="25.4" x2="53.34" y2="22.86" width="0.254" layer="1"/>
+<wire x1="53.34" y1="22.86" x2="53.34" y2="19.05" width="0.254" layer="1"/>
 </signal>
 <signal name="N$9">
@@
 <wire x1="66.04" y1="11.43" x2="64.135" y2="13.335" width="0.254" layer="1"/>
 <wire x1="64.135" y1="13.335" x2="46.99" y2="13.335" width="0.254" layer="1"/>
-<wire x1="40.64" y1="13.97" x2="46.355" y2="13.97" width="0.254" layer="1"/>
+<wire x1="41.91" y1="13.97" x2="46.355" y2="13.97" width="0.254" layer="1"/>
 </signal>
 <signal name="VCC">
@@
 <wire x1="24.13" y1="24.13" x2="26.67" y2="24.13" width="0.4064" layer="1"/>
 <wire x1="29.21" y1="33.02" x2="26.67" y2="33.02" width="0.4064" layer="1"/>
-<wire x1="26.67" y1="24.13" x2="31.75" y2="24.13" width="0.4064" layer="1"/>
-<wire x1="31.75" y1="24.13" x2="36.83" y2="29.21" width="0.4064" layer="1"/>
-<wire x1="36.83" y1="29.21" x2="41.91" y2="29.21" width="0.4064" layer="1"/>
+<wire x1="26.67" y1="24.13" x2="32.22625" y2="24.13" width="0.4064" layer="1"/>
+<wire x1="32.22625" y1="24.13" x2="36.29025" y2="29.21" width="0.4064" layer="1"/>
+<wire x1="36.29025" y1="29.21" x2="41.91" y2="29.21" width="0.4064" layer="1"/>
 <wire x1="41.91" y1="29.21" x2="44.45" y2="26.67" width="0.4064" layer="1"/>
 <wire x1="19.05" y1="29.21" x2="19.05" y2="31.75" width="0.4064" layer="1"/>
