File: 8Bit-audio-v2/8Bit-audio-7524-axelb-v2.sch (EAGLE design)
At the start: 21 parts, among them IC1 LM358 or MCP6022, IC4 AD7524LN, X1 AUX 3,5mm

Commit message: New footprints
Parts:
- C1, C2, C6: device rcl:CPOL-EUE5-5 -> myLbr:CPOL-EUE2.5-7
Connections:
- net AUX: now also C6.-2
- net GND: now also C1.-2
- net N$3: now also C2.-2
Changed lines of the file:
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@@
 <setting verticaltext="up"/>
 </settings>
-<grid distance="0.1" unitdist="inch" unit="mil" style="lines" multiple="1" display="yes" altdistance="12.5" altunitdist="mil" altunit="mil"/>
+<grid distance="0.1" unitdist="inch" unit="inch" style="lines" multiple="1" display="no" altdistance="0.01" altunitdist="inch" altunit="inch"/>
 <layers>
 <layer number="1" name="Top" color="4" fill="1" visible="no" active="no"/>
@@
 <part name="IC1" library="linear" library_urn="urn:adsk.eagle:library:262" deviceset="LM358" device="N" package3d_urn="urn:adsk.eagle:package:16409/2" value="LM358 or MCP6022"/>
 <part name="L1" library="rcl" library_urn="urn:adsk.eagle:library:334" deviceset="L-EU" device="0207/10" package3d_urn="urn:adsk.eagle:package:23491/2" value="1mH"/>
-<part name="C1" library="rcl" library_urn="urn:adsk.eagle:library:334" deviceset="CPOL-EU" device="E5-5" package3d_urn="urn:adsk.eagle:package:23367/2" value="100µ"/>
+<part name="C1" library="myLbr" deviceset="CPOL-EU" device="E2.5-7" value="100µ"/>
 <part name="JP1" library="pinhead" library_urn="urn:adsk.eagle:library:325" deviceset="PINHD-1X13" device="" package3d_urn="urn:adsk.eagle:package:22421/2" value="DATA"/>
 <part name="JP2" library="pinhead" library_urn="urn:adsk.eagle:library:325" deviceset="PINHD-1X1" device="" package3d_urn="urn:adsk.eagle:package:22485/2" value="TP1"/>
 <part name="R1" library="rcl" library_urn="urn:adsk.eagle:library:334" deviceset="R-EU_" device="0207/10" package3d_urn="urn:adsk.eagle:package:23491/2" value="100k"/>
 <part name="R2" library="rcl" library_urn="urn:adsk.eagle:library:334" deviceset="R-EU_" device="0207/10" package3d_urn="urn:adsk.eagle:package:23491/2" value="100k"/>
-<part name="C2" library="rcl" library_urn="urn:adsk.eagle:library:334" deviceset="CPOL-EU" device="E5-5" package3d_urn="urn:adsk.eagle:package:23367/2" value="1µ"/>
+<part name="C2" library="myLbr" deviceset="CPOL-EU" device="E2.5-7" value="1µ"/>
 <part name="R3" library="rcl" library_urn="urn:adsk.eagle:library:334" deviceset="R-EU_" device="0207/10" package3d_urn="urn:adsk.eagle:package:23491/2" value="10k"/>
 <part name="R4" library="rcl" library_urn="urn:adsk.eagle:library:334" deviceset="R-EU_" device="0207/10" package3d_urn="urn:adsk.eagle:package:23491/2" value="220k"/>
@@
 <part name="C4" library="myLbr" deviceset="RCL_C-EU" device="025_050-055X075" value="1nF"/>
 <part name="C5" library="myLbr" deviceset="RCL_C-EU" device="025_050-055X075" value="47pF"/>
-<part name="C6" library="rcl" library_urn="urn:adsk.eagle:library:334" deviceset="CPOL-EU" device="E5-5" package3d_urn="urn:adsk.eagle:package:23367/2" value="100µ"/>
+<part name="C6" library="myLbr" deviceset="CPOL-EU" device="E2.5-7" value="100µ"/>
 <part name="P+3" library="supply1" deviceset="VCC" device=""/>
 <part name="R6" library="myLbr" deviceset="POT_3RP/1610N" device="" value="10k"/>
@@
 <wire x1="149.86" y1="60.96" x2="147.32" y2="60.96" width="0.1524" layer="91"/>
 <junction x="149.86" y="55.88"/>
+<pinref part="C6" gate="G$1" pin="-2"/>
+<junction x="147.32" y="60.96"/>
 </segment>
 </net>
@@
 <junction x="-35.56" y="53.34"/>
 <label x="-56.134" y="52.324" size="1.778" layer="95"/>
+<pinref part="C1" gate="G$1" pin="-2"/>
+<junction x="22.86" y="58.42"/>
 </segment>
 </net>
@@
 <pinref part="R1" gate="G$1" pin="2"/>
 <wire x1="68.58" y1="63.5" x2="68.58" y2="66.04" width="0.1524" layer="91"/>
-</segment>
-</net>
+<pinref part="C2" gate="G$1" pin="-2"/>
+<junction x="66.04" y="63.5"/>
+</segment>
+</net>
